File: hardware/logicboard/sc-001.brd (EAGLE design)
At the start: 72 x 42 mm, 14 parts, among them Q1 60V/32A/35mΩ, Q2 60V/32A/35mΩ, Q3 60V/32A/35mΩ, Q4 60V/32A/35mΩ

Commit message: Ext DC port.
Parts:
- added J1: (no value), con-jack:SPC4077
- added S1: 9077-1, switch-misc:9077-1
- moved C1 16.3 mm to (30.0, 15.0)
- moved SV1 6.00 mm to (42.0, 11.0)
Connections:
- new net V+: J1.3, S1.1
- new net VCC/3: C1.1, D1.C, D2.C, D3.C, D4.C, R1.1, S1.2, SV2.12, SV2.16, SV2.4, SV2.8
- net GND: now also J1.1, J1.2
- net VCC/2: now also S1.3; no longer C1.1, D1.C, D2.C, D3.C, D4.C, R1.1, SV2.12, SV2.16, SV2.4, SV2.8
Routing:
- net VCC/3: track 0.00 -> 95.7 mm
- net VCC/2: track 113.0 -> 51.2 mm
- net V+: track 0.00 -> 16.2 mm
- net GND: track 114.4 -> 123.2 mm
- net DTCT3: track 27.8 -> 21.6 mm
- net ANLG2: track 24.2 -> 18.1 mm
- net DTCT0: track 36.1 -> 41.5 mm
- net ANLG1: track 21.4 -> 25.7 mm
- net DTCT1: track 20.1 -> 24.1 mm
- net ANLG3: track 35.0 -> 37.7 mm
- net DRVR0: track 20.6 -> 22.4 mm
- net DTCT2: track 13.2 -> 11.8 mm
Other:
- board text added: "V+"
- board text added: "V/2"
